File: 00-proyecto-2/grupo-01/esquematicos/version-1/proyecto-2-grupo01.kicad_sch (KiCad schematic)
At the start: 17 parts, among them SW1 RotaryEncoder_Switch, SW2 SW_Push

Commit message: add and test 50n1d0-v05
Connections:
- net LOOP is gone; now on net BOTON: R6.1, SW2.1
- net GND: now also SW1.C, SW1.S2; no longer SW1.GND
- net GIRO A: now reaches A1.14 (GPIO10)
- net GIRO A: now also SW1.A
- net GIRO B: now reaches A1.15 (GPIO11)
- net GIRO B: now also SW1.B
- net CLOCK: no longer names the net of A1.19 (GPIO14)
- net CLOCK: no longer SW1.CLK
- net DT: no longer names the net of A1.20 (GPIO15)
- net SELECTOR renamed PULSADOR ENCODER
- net PULSADOR ENCODER: now also SW1.S1; no longer SW1.SW
- removed net SW: SW1.DT
- removed net VCC: SW1.VCC
Other:
- note added: "Encoder rotatorio KY-040 360 grados Se desplaza a través del menú de sonidos"
- note added: "INPUTS"
- note added: "OUTPUTS"
- note removed: "ENTRADAS"
- note removed: "Encoder rotatorio KY-040 360 grados"
- note removed: "No es relevante el valor del pote"
- note removed: "SALIDAS"
- note removed: "Se desplaza a través del menú de sonidos"
- note removed: "Solo debe ser lineal / tipo B"
- moved on the sheet: RV1
